File: RP2040_Macropad.kicad_pcb (KiCad board)
At the start: 2 copper layers, 54 parts, among them J1 External GPIOs, SW1 SW_Push, SW10 RotaryEncoder_Switch, SW11 SW_Push, SW12 SW_Push, SW2 SW_Push, SW3 SW_Push, SW4 SW_Push, SW5 SW_Push, SW6 SW_Push, SW7 SW_Push, SW8 SW_Push, SW9 SW_Push, U1 kb2040

Commit message: layout complete
Parts:
- removed D13, D14, D15, D16, D17, D18, D19: SK6812MINI, LED_SMD:LED_SK6812MINI_PLCC4_3.5x3.5mm_P1.75mm
- removed D20, D22: 1N4148W, Diode_SMD:D_SOD-123
- removed J1: External GPIOs, Connector_PinHeader_2.54mm:PinHeader_1x04_P2.54mm_Vertical
- removed R1, R2, R3, R4: 10k, Resistor_SMD:R_0603_1608Metric
- added H1: MountingHole_Pad, MountingHole:MountingHole_3.2mm_M3_DIN965_Pad, F.Cu at (108.0, 26.7)
- added H2: MountingHole_Pad, MountingHole:MountingHole_3.2mm_M3_DIN965_Pad, F.Cu at (108.0, 106.0)
- added H3: MountingHole_Pad, MountingHole:MountingHole_3.2mm_M3_DIN965_Pad, F.Cu at (28.6, 26.7)
- added H4: MountingHole_Pad, MountingHole:MountingHole_3.2mm_M3_DIN965_Pad, F.Cu at (28.6, 106.0)
- added LED1: MX_SK6812MINI-E, PCM_marbastlib-mx:LED_MX_6028R, B.Cu at (57.1, 43.2)
- added LED10: MX_SK6812MINI-E, PCM_marbastlib-mx:LED_MX_6028R, B.Cu at (57.1, 100.3)
- added LED11: MX_SK6812MINI-E, PCM_marbastlib-mx:LED_MX_6028R, B.Cu at (76.2, 100.3)
- added LED2: MX_SK6812MINI-E, PCM_marbastlib-mx:LED_MX_6028R, B.Cu at (38.1, 43.2)
- added LED3: MX_SK6812MINI-E, PCM_marbastlib-mx:LED_MX_6028R, B.Cu at (38.1, 62.2)
- added LED4: MX_SK6812MINI-E, PCM_marbastlib-mx:LED_MX_6028R, B.Cu at (57.1, 62.2)
- added LED5: MX_SK6812MINI-E, PCM_marbastlib-mx:LED_MX_6028R, B.Cu at (76.2, 62.2)
- added LED6: MX_SK6812MINI-E, PCM_marbastlib-mx:LED_MX_6028R, B.Cu at (76.2, 81.3)
- added LED7: MX_SK6812MINI-E, PCM_marbastlib-mx:LED_MX_6028R, B.Cu at (38.1, 100.3)
- added LED8: MX_SK6812MINI-E, PCM_marbastlib-mx:LED_MX_6028R, B.Cu at (38.1, 81.3)
- added LED9: MX_SK6812MINI-E, PCM_marbastlib-mx:LED_MX_6028R, B.Cu at (57.1, 81.3)
- C1, C2: value 10n -> 100nf; moved to B.Cu
- C10, C11, C3, C4, C5, C6, C7, C8, C9, D1, D10, D2, D3, D4, D5, D6, D7, D8, D9, R5, R7, R8: moved to B.Cu
- D11, D12: value SK6812MINI -> 1N4148W; footprint LED_SMD:LED_SK6812MINI_PLCC4_3.5x3.5mm_P1.75mm -> Diode_SMD:D_SOD-123; moved to B.Cu
- SW10: value RotaryEncoder_Switch -> SW_Push; footprint Rotary_Encoder:RotaryEncoder_Alps_EC11E-Switch_Vertical_H20mm -> PCM_Switch_Keyboard_Hotswap_Kailh:SW_Hotswap_Kailh_MX_1.00u
- SW3: value SW_Push -> RotaryEncoder_Switch; footprint PCM_Switch_Keyboard_Hotswap_Kailh:SW_Hotswap_Kailh_MX_1.00u -> Rotary_Encoder:RotaryEncoder_Alps_EC11E-Switch_Vertical_H20mm
- moved D1 196.2 mm to (43.2, 41.9), turned to 90 degrees
- moved D4 195.8 mm to (43.2, 61.0), turned to 90 degrees
- moved D7 195.8 mm to (43.2, 80.0), turned to 90 degrees
- moved C1 185.3 mm to (39.4, 46.4)
- moved C3 182.3 mm to (39.4, 65.4)
- moved C6 180.6 mm to (39.4, 84.5)
- moved C7 179.5 mm to (39.4, 103.5)
- moved D2 177.5 mm to (62.2, 41.9), turned to 90 degrees
- moved D5 176.9 mm to (62.2, 61.0), turned to 90 degrees
- moved D8 176.7 mm to (62.2, 80.0), turned to 90 degrees
- moved C2 167.6 mm to (58.4, 46.4)
- moved C9 164.8 mm to (58.4, 84.5)
- moved C10 164.5 mm to (58.4, 103.5)
- moved C4 164.1 mm to (58.4, 65.4)
- moved D3 159.1 mm to (81.3, 41.1), turned to 90 degrees
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Connections:
- C1 pad 2: Enocder A -> +3.3V
- C10 pad 2: 3.3V -> +3.3V
- C11 pad 2: 3.3V -> +3.3V
- C2 pad 2: Enocder B -> +3.3V
- C3 pad 2: 3.3V -> +3.3V
- C4 pad 2: 3.3V -> +3.3V
- C5 pad 2: 3.3V -> +3.3V
- C6 pad 2: 3.3V -> +3.3V
- C7 pad 2: 3.3V -> +3.3V
- C8 pad 2: 3.3V -> +3.3V
- C9 pad 2: 3.3V -> +3.3V
- D1 pad 1: Row 0 -> Row 1
- D10 pad 1: GND -> Row 4
- D11 pad 1: Net-(D11-DOUT) -> Row 4
- D11 pad 2: GND -> Net-(D11-A)
- D12 pad 1: Net-(D12-DOUT) -> Row 4
- D12 pad 2: GND -> Net-(D12-A)
- D2 pad 1: Row 0 -> Row 1
- D4 pad 1: Row 1 -> Row 2
- D5 pad 1: Row 1 -> Row 2
- D7 pad 1: Row 2 -> Row 3
- D8 pad 1: Row 2 -> Row 3
- D9 pad 1: GND -> Row 3
- R5 pad 2: Net-(D11-DIN) -> Net-(LED1-DIN)
- R7 pad 1: 3.3V -> +3.3V
- R8 pad 1: 3.3V -> +3.3V
- SSD1306 pad 3: 3.3V -> +3.3V
- SW1 pad 1: Col 0 -> Col 1
- SW1 pad 2: Net-(D22-A) -> Net-(D1-A)
- SW11 pad 1: Solo Key 1 -> Col 2
- SW11 pad 2: Net-(D9-A) -> Net-(D11-A)
- SW12 pad 1: Solo Key 2 -> Col 3
- SW12 pad 2: Net-(D10-A) -> Net-(D12-A)
- SW2 pad 1: Col 1 -> Col 2
- SW2 pad 2: Net-(D1-A) -> Net-(D2-A)
- SW4 pad 1: Col 0 -> Col 1
- SW4 pad 2: Net-(D3-A) -> Net-(D4-A)
- SW5 pad 1: Col 1 -> Col 2
- SW5 pad 2: Net-(D4-A) -> Net-(D5-A)
- SW6 pad 1: Col 2 -> Col 3
- SW6 pad 2: Net-(D5-A) -> Net-(D6-A)
- SW7 pad 1: Col 0 -> Col 1
- SW7 pad 2: Net-(D6-A) -> Net-(D7-A)
- SW8 pad 1: Col 1 -> Col 2
- SW8 pad 2: Net-(D7-A) -> Net-(D8-A)
- SW9 pad 1: Col 2 -> Col 3
- SW9 pad 2: Net-(D8-A) -> Net-(D9-A)
- U1 pad 10: Row 2 -> Row 3
- U1 pad 11: Row 3 -> Row 4
- U1 pad 12: Enocder A -> D8
- U1 pad 13: Enocder B -> D9
- U1 pad 18: 3.3V -> +3.3V
- U1 pad 3: Col 0 -> Col 1
- U1 pad 6: Col 1 -> Col 2
- U1 pad 7: Col 2 -> Col 3
- U1 pad 8: Row 0 -> Row 1
- U1 pad 9: Row 1 -> Row 2
Routing:
- net Col 1: track 0.00 -> 57.1 mm
- net GND: track 42.7 -> 0.00 mm
- net Net-(D2-A): track 0.00 -> 9.47 mm
- net Net-(D11-A): track 0.00 -> 9.47 mm
- net Net-(D8-A): track 0.00 -> 9.47 mm
- net Net-(D6-A): track 0.00 -> 9.47 mm
- net Net-(D4-A): track 0.00 -> 9.47 mm
- net Net-(D9-A): track 0.00 -> 9.47 mm
- net Net-(D12-A): track 0.00 -> 9.47 mm
- net Net-(D1-A): track 0.00 -> 9.47 mm
- net Net-(D7-A): track 0.00 -> 9.47 mm
- net Net-(D10-A): track 0.00 -> 9.47 mm
- net Net-(D5-A): track 0.00 -> 9.36 mm
Other:
- board outline added: 86.2 x 86.4 mm
